File: PCB/SerialGamePad.sch (KiCad schematic (older format))
At the start: 14 parts, among them P0 CONN_01X02, P1 CONN_01X02, P2 CONN_01X02, P3 CONN_01X02, P4 CONN_01X02, P5 CONN_01X02

Commit message: fixing autosaves
Parts:
- C1: footprint (none) -> w_capacitors:CP_6.3x11mm
Changed lines of the file:
@@
 F 0 "C1" H 4875 5150 50  0000 L CNN
 F 1 "CP1" H 4875 4950 50  0000 L CNN
-F 2 "" H 4850 5050 60  0000 C CNN
+F 2 "w_capacitors:CP_6.3x11mm" H 4850 5050 60  0001 C CNN
 F 3 "" H 4850 5050 60  0000 C CNN
 	1    4850 5050
